File: Hardware/PCB/joystick/joystick.kicad_pcb (KiCad board)
At the start: 2 copper layers, 94 x 107 mm, 57 parts, among them J1 Synth_power_2x5, J11 AudioJack2, J12 3_pin_Molex_header, J13 AudioJack2, J14 2_pin_Molex_header, J4 AudioJack2, J5 6 pin Molex header, J6 AudioJack2, J7 3_pin_Molex_header, J8 2_pin_Molex_header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

Commit message: KiCad 6
Connections:
- net /Y channel/~YOUT renamed /Y channel/~{YOUT}
- net /~XOUT renamed /~{XOUT}
Other:
- net class Default removed
- net class Power removed
